Commit message: handy bridge complete

File: handy_ros2/urdf/robot.urdf (robot description, URDF)
Before this commit: robot C:\Users\david\Documents\Code\handy\software\urdf, 9 links, 8 joints
Links:
- link base: geometry collision mesh filename=package://handy_ros2/urdf/assets/base.stl; collision mesh filename=package://handy_ros2/urdf/assets/part_1.stl
- link encoder_link_assembly: geometry collision mesh filename=package://handy_ros2/urdf/assets/57155k526_stainless_steel_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; collision mesh filename=package://handy_ros2/urdf/assets/57155k526_stainless_steel_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
- link encoder_link_assembly_2: geometry collision mesh filename=package://handy_ros2/urdf/assets/57155k526_stainless_steel_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; collision mesh filename=package://handy_ros2/urdf/assets/57155k526_stainless_steel_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
- link part_1: geometry collision mesh filename=package://handy_ros2/urdf/assets/part_1__3.stl; visual mesh filename=package://handy_ros2/urdf/assets/part_1__3.stl
- link part_1_2: geometry collision mesh filename=package://handy_ros2/urdf/assets/part_1__3.stl; visual mesh filename=package://handy_ros2/urdf/assets/part_1__3.stl
- link part_2: geometry collision mesh filename=package://handy_ros2/urdf/assets/part_2.stl; visual mesh filename=package://handy_ros2/urdf/assets/part_2.stl
- link passive_link_assembly__configuration_default: geometry collision mesh filename=package://handy_ros2/urdf/assets/m2x2_5_insert.stl; collision mesh filename=package://handy_ros2/urdf/assets/m2x2_5_insert.stl
- link passive_link_assembly__configuration_thumb: geometry collision mesh filename=package://handy_ros2/urdf/assets/m2x2_5_insert.stl; collision mesh filename=package://handy_ros2/urdf/assets/m2x2_5_insert.stl
Joints:
- removed joint index_3
- removed joint thumb_4
- added joint index_2: type revolute, parent passive_link_assembly__configuration_default, child part_1, origin xyz=-0.045 3.46945e-18 3.46945e-18 rpy=-3.14159 -1.84264e-47 0, axis 0 0 1, limit lower=-3.141592653589793 upper=3.141592653589793 effort=10 velocity=10
- added joint thumb_2: type revolute, parent passive_link_assembly__configuration_thumb, child part_1_2, origin xyz=-0.055 -6.93889e-18 -6.07153e-18 rpy=3.14159 -5.55112e-17 3.55596e-14, axis 0 0 1, limit lower=-3.141592653589793 upper=3.141592653589793 effort=10 velocity=10
- joint index_1: origin xyz=-0.06 -1.04083e-17 0 rpy=3.14159 1.10559e-47 1.01465e-17 -> xyz=-0.06 -1.38778e-17 0 rpy=3.14159 1.10559e-47 0
- joint thumb_1: origin xyz=0.06 0 -2.60209e-18 rpy=-3.14159 1.62548e-16 3.14159 -> xyz=0.06 0 8.67362e-19 rpy=-3.14159 2.22045e-16 3.14159
- joint thumb_3: child part_1_2 -> part_2; origin xyz=-0.055 -6.93889e-18 -1.21431e-17 rpy=3.14159 -3.66515e-17 3.55596e-14 -> xyz=0.0335773 0.0457111 -0.007 rpy=-1.5708 -0 1.5708; parent passive_link_assembly__configuration_thumb -> base

Commit message: imu integration

File: handy_ros2/urdf/robot.urdf (robot description, URDF)
Before this commit: robot urdf, 9 links, 8 joints
Links:
- added link index_tip, mass 1e-9
- added link thumb_tip, mass 1e-9
Joints:
- added joint index_tip_frame: type fixed, parent part_1, child index_tip, origin xyz=-0.0207217 0.02 7.5e-05 rpy=-1.5708 -0 0, axis 0 0 0
- added joint thumb_tip_frame: type fixed, parent part_1_2, child thumb_tip, origin xyz=-0.0207217 -0.02 7.5e-05 rpy=1.5708 -5.55112e-17 3.15544e-30, axis 0 0 0

Commit message: added pinky

File: handy_ros2/urdf/robot.urdf (robot description, URDF)
Before this commit: robot urdf, 11 links, 10 joints
Links:
- removed link encoder_link_assembly
- removed link encoder_link_assembly_2
- added link encoder_link_assembly__configuration_default, mass 0.000597845; collision mesh filename=package://handy_ros2/urdf/assets/57155k526_stainless_steel_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; collision mesh filename=package://handy_ros2/urdf/assets/57155k526_stainless_steel_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
- added link encoder_link_assembly__configuration_default_2, mass 0.000597845; collision mesh filename=package://handy_ros2/urdf/assets/57155k526_stainless_steel_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; collision mesh filename=package://handy_ros2/urdf/assets/57155k526_stainless_steel_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
- added link encoder_link_assembly__configuration_default_3, mass 0.000597845; collision mesh filename=package://handy_ros2/urdf/assets/57155k526_stainless_steel_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; collision mesh filename=package://handy_ros2/urdf/assets/57155k526_stainless_steel_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
- added link part_1_3, mass 1e-09; collision mesh filename=package://handy_ros2/urdf/assets/part_1__2.stl; visual mesh filename=package://handy_ros2/urdf/assets/part_1__2.stl
- added link passive_link_assembly__configuration_pinky, mass 1e-09; collision mesh filename=package://handy_ros2/urdf/assets/m2x2_5_insert.stl; collision mesh filename=package://handy_ros2/urdf/assets/m2x2_5_insert.stl
- added link pinky_tip, mass 1e-9
- link base: geometry collision mesh filename=package://handy_ros2/urdf/assets/base.stl; collision mesh filename=package://handy_ros2/urdf/assets/part_1.stl
- link part_1: geometry collision mesh filename=package://handy_ros2/urdf/assets/part_1__2.stl; visual mesh filename=package://handy_ros2/urdf/assets/part_1__2.stl
- link part_1_2: geometry collision mesh filename=package://handy_ros2/urdf/assets/part_1__2.stl; visual mesh filename=package://handy_ros2/urdf/assets/part_1__2.stl
Joints:
- added joint pinky_0: type revolute, parent base, child encoder_link_assembly__configuration_default_3, origin xyz=-0.0289227 -0.0367889 0.0136569 rpy=-1.5708 0.785398 1.5708, axis 0 0 1, limit lower=-3.141592653589793 upper=3.141592653589793 effort=10 velocity=10
- added joint pinky_1: type revolute, parent encoder_link_assembly__configuration_default_3, child passive_link_assembly__configuration_pinky, origin xyz=-0.06 1.04083e-17 4.875e-05 rpy=-3.14159 -5.55112e-17 6.66134e-16, axis 0 0 1, limit lower=-3.141592653589793 upper=3.141592653589793 effort=10 velocity=10
- added joint pinky_2: type revolute, parent passive_link_assembly__configuration_pinky, child part_1_3, origin xyz=-0.03 3.1225e-17 1.04083e-17 rpy=-5.55112e-17 5.55112e-17 6.66134e-16, axis 0 0 1, limit lower=-3.141592653589793 upper=3.141592653589793 effort=10 velocity=10
- added joint pinky_tip_frame: type fixed, parent part_1_3, child pinky_tip, origin xyz=-0.0207217 0.02 7.5e-05 rpy=-1.5708 6.16298e-33 0, axis 0 0 0
- joint index_0: child encoder_link_assembly -> encoder_link_assembly__configuration_default
- joint index_1: parent encoder_link_assembly -> encoder_link_assembly__configuration_default
- joint thumb_0: child encoder_link_assembly_2 -> encoder_link_assembly__configuration_default_2
- joint thumb_1: parent encoder_link_assembly_2 -> encoder_link_assembly__configuration_default_2
